File: Eagle/Asistente_Alzhaimer.sch (EAGLE design)
At the start: 10 parts, among them Q1 2N3904

Commit message: SCH con ESP32 al 50%
Parts:
- removed HC-05: (no value), con-lsta:FE06-1
- added MOD2: WIRELESS-BLUETOOTH-HC-05, diy-modules:WIRELESS-BLUETOOTH-HC-05
- added S1: (no value), adafruit:40-XX-ROUND
- MOD1: value ARDUINO_MKR1000 -> ESP32_DEVKIT_V1; device Circuitos-Creativos-Modulos:ARDUINO_MKR1000 -> Circuitos-Creativos-Modulos:ESP32_DEVKIT_V1
- R1: value 330R -> 1k
- R3: value 2k2 -> 1k
Connections:
- removed net LED1: R1.1
- new net +3V3: LCD1.VCC, MOD1.3V3
- new net BL: MOD1.D21/SDA
- new net BOT-PANIC: MOD1.D14/ADC2_6
- new net CE: MOD1.D4/ADC2_0
- new net CLK: MOD1.D19/MISO
- new net DC: MOD1.D5
- new net DIN: MOD1.D18/SCK
- new net LED: MOD1.D27/ADC2_7, R1.1
- new net RST: MOD1.D2/ADC2_2
- new net RXD2: MOD1.D16/RX2
- new net STATE: MOD1.D15/ADC2_3
- new net TXD2: MOD1.D17/TX2
- net +5V: now also MOD1.VIN
- net BUZZ: now also MOD1.D26/ADC2_9
- net GND: now also LCD1.GND, MOD1.GND, MOD1.GND1
Changed lines of the file:
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@@
 <parts>
 <part name="U$1" library="Circuitos-Creativos-Estilos" deviceset="A4_HORIZONTAL" device=""/>
-<part name="MOD1" library="Circuitos-Creativos-Modulos" deviceset="ARDUINO_MKR1000" device=""/>
 <part name="X1" library="con-ptr500" deviceset="AK500/2" device=""/>
 <part name="P+1" library="supply1" deviceset="+5V" device=""/>
@@
 <part name="BUZZER" library="buzzer" deviceset="F/CM12P" device=""/>
 <part name="Q1" library="Ingenialo" deviceset="2N3904" device=""/>
-<part name="R3" library="rcl" deviceset="R-US_" device="0204/7" value="2k2"/>
+<part name="R3" library="rcl" deviceset="R-US_" device="0204/7" value="1k"/>
 <part name="GND19" library="supply1" deviceset="GND" device=""/>
-<part name="R1" library="rcl" deviceset="R-US_" device="0204/7" value="330R"/>
+<part name="R1" library="rcl" deviceset="R-US_" device="0204/7" value="1k"/>
 <part name="LED1" library="led" deviceset="LED" device="3MM" value="ALARMA"/>
 <part name="GND2" library="supply1" deviceset="GND" device=""/>
 <part name="P+2" library="supply1" deviceset="+5V" device=""/>
-<part name="HC-05" library="con-lsta" deviceset="FE06-1" device=""/>
+<part name="MOD1" library="Circuitos-Creativos-Modulos" deviceset="ESP32_DEVKIT_V1" device=""/>
+<part name="GND3" library="supply1" deviceset="GND" device=""/>
+<part name="MOD2" library="diy-modules" deviceset="WIRELESS-BLUETOOTH-HC-05" device=""/>
+<part name="GND4" library="supply1" deviceset="GND" device=""/>
+<part name="+3V2" library="supply1" deviceset="+3V3" device=""/>
+<part name="S1" library="adafruit" deviceset="40-XX" device="-ROUND"/>
 </parts>
 <sheets>
@@
 <attribute name="SHEET" x="186.055" y="1.27" size="2.54" layer="94"/>
 </instance>
-<instance part="MOD1" gate="G$1" x="53.34" y="116.84" smashed="yes">
-<attribute name="NAME" x="37.084" y="146.304" size="1.778" layer="95"/>
-<attribute name="VALUE" x="40.132" y="77.47" size="1.778" layer="96"/>
-</instance>
 <instance part="X1" gate="-1" x="124.46" y="114.3" smashed="yes">
 <attribute name="NAME" x="123.19" y="115.189" size="1.778" layer="95" rot="R180"/>
@@
 <attribute name="VALUE" x="120.65" y="105.537" size="1.778" layer="96"/>
 </instance>
-<instance part="P+1" gate="1" x="104.14" y="83.82" smashed="yes">
-<attribute name="VALUE" x="101.6" y="78.74" size="1.778" layer="96" rot="R90"/>
-</instance>
-<instance part="GND1" gate="1" x="91.44" y="73.66" smashed="yes">
-<attribute name="VALUE" x="88.9" y="71.12" size="1.778" layer="96"/>
-</instance>
-<instance part="+3V1" gate="G$1" x="104.14" y="116.84" smashed="yes">
-<attribute name="VALUE" x="101.6" y="111.76" size="1.778" layer="96" rot="R90"/>
+<instance part="P+1" gate="1" x="73.66" y="129.54" smashed="yes">
+<attribute name="VALUE" x="76.2" y="132.08" size="1.778" layer="96" rot="R180"/>
+</instance>
+<instance part="GND1" gate="1" x="78.74" y="121.92" smashed="yes" rot="R90">
+<attribute name="VALUE" x="81.28" y="119.38" size="1.778" layer="96" rot="R90"/>
+</instance>
+<instance part="+3V1" gate="G$1" x="17.78" y="129.54" smashed="yes">
+<attribute name="VALUE" x="20.32" y="132.08" size="1.778" layer="96" rot="R180"/>
 </instance>
 <instance part="LCD1" gate="G$1" x="142.24" y="139.7" smashed="yes">
@@
 <attribute name="VALUE" x="147.32" y="78.74" size="1.778" layer="96" rot="R180"/>
 </instance>
-<instance part="HC-05" gate="G$1" x="198.12" y="119.38" smashed="yes">
-<attribute name="VALUE" x="196.85" y="109.22" size="1.778" layer="96"/>
-<attribute name="NAME" x="196.85" y="130.302" size="1.778" layer="95"/>
-</instance>
+<instance part="MOD1" gate="G$1" x="45.72" y="106.68" smashed="yes">
+<attribute name="NAME" x="28.956" y="138.43" size="1.778" layer="95"/>
+<attribute name="VALUE" x="34.29" y="75.946" size="1.778" layer="96"/>
+</instance>
+<instance part="GND3" gate="1" x="7.62" y="121.92" smashed="yes" rot="R270">
+<attribute name="VALUE" x="5.08" y="124.46" size="1.778" layer="96" rot="R270"/>
+</instance>
+<instance part="MOD2" gate="G$1" x="104.14" y="86.36" smashed="yes">
+<attribute name="NAME" x="106.68" y="96.52" size="1.778" layer="95" rot="R180"/>
+<attribute name="VALUE" x="88.9" y="73.66" size="1.778" layer="96"/>
+</instance>
+<instance part="GND4" gate="1" x="157.48" y="114.3" smashed="yes">
+<attribute name="VALUE" x="154.94" y="111.76" size="1.778" layer="96"/>
+</instance>
+<instance part="+3V2" gate="G$1" x="147.32" y="111.76" smashed="yes" rot="R180">
+<attribute name="VALUE" x="144.78" y="109.22" size="1.778" layer="96"/>
+</instance>
+<instance part="S1" gate="1" x="96.52" y="50.8"/>
 </instances>
 <busses>
@@
 <wire x1="198.12" y1="53.34" x2="198.12" y2="48.26" width="0.1524" layer="91"/>
 </segment>
+<segment>
+<pinref part="GND3" gate="1" pin="GND"/>
+<pinref part="MOD1" gate="G$1" pin="GND"/>
+<wire x1="10.16" y1="121.92" x2="22.86" y2="121.92" width="0.1524" layer="91"/>
+</segment>
+<segment>
+<pinref part="GND1" gate="1" pin="GND"/>
+<pinref part="MOD1" gate="G$1" pin="GND1"/>
+<wire x1="76.2" y1="121.92" x2="68.58" y2="121.92" width="0.1524" layer="91"/>
+</segment>
+<segment>
+<pinref part="LCD1" gate="G$1" pin="GND"/>
+<wire x1="152.4" y1="121.92" x2="152.4" y2="119.38" width="0.1524" layer="91"/>
+<wire x1="152.4" y1="119.38" x2="157.48" y2="119.38" width="0.1524" layer="91"/>
+<pinref part="GND4" gate="1" pin="GND"/>
+<wire x1="157.48" y1="119.38" x2="157.48" y2="116.84" width="0.1524" layer="91"/>
+</segment>
 </net>
 <net name="N$7" class="0">
@@
 <wire x1="144.78" y1="73.66" x2="144.78" y2="71.12" width="0.1524" layer="91"/>
 </segment>
+<segment>
+<pinref part="MOD1" gate="G$1" pin="VIN"/>
+<pinref part="P+1" gate="1" pin="+5V"/>
+<wire x1="68.58" y1="124.46" x2="73.66" y2="124.46" width="0.1524" layer="91"/>
+<wire x1="73.66" y1="124.46" x2="73.66" y2="127" width="0.1524" layer="91"/>
+</segment>
 </net>
 <net name="BUZZ" class="0">
@@
 <label x="124.46" y="55.88" size="1.27" layer="95" rot="R180" xref="yes"/>
 </segment>
-</net>
-<net name="LED1" class="0">
+<segment>
+<pinref part="MOD1" gate="G$1" pin="D26/ADC2_9"/>
+<wire x1="68.58" y1="109.22" x2="71.12" y2="109.22" width="0.1524" layer="91"/>
+<label x="71.12" y="109.22" size="1.27" layer="95" ratio="10" xref="yes"/>
+</segment>
+</net>
+<net name="LED" class="0">
 <segment>
 <pinref part="R1" gate="G$1" pin="1"/>
@@
 <label x="190.5" y="76.2" size="1.27" layer="95" rot="R180" xref="yes"/>
 </segment>
-</net>
+<segment>
+<pinref part="MOD1" gate="G$1" pin="D27/ADC2_7"/>
+<wire x1="68.58" y1="111.76" x2="71.12" y2="111.76" width="0.1524" layer="91"/>
+<label x="71.12" y="111.76" size="1.27" layer="95" ratio="10" xref="yes"/>
+</segment>
+</net>
+<net name="+3V3" class="0">
+<segment>
+<pinref part="MOD1" gate="G$1" pin="3V3"/>
+<pinref part="+3V1" gate="G$1" pin="+3V3"/>
+<wire x1="22.86" y1="124.46" x2="17.78" y2="124.46" width="0.1524" layer="91"/>
+<wire x1="17.78" y1="124.46" x2="17.78" y2="127" width="0.1524" layer="91"/>
+</segment>
+<segment>
+<pinref part="LCD1" gate="G$1" pin="VCC"/>
+<pinref part="+3V2" gate="G$1" pin="+3V3"/>
+<wire x1="147.32" y1="114.3" x2="147.32" y2="121.92" width="0.1524" layer="91"/>
+</segment>
+</net>
+<net name="RST" class="0">
+<segment>
+<pinref part="MOD1" gate="G$1" pin="D2/ADC2_2"/>
+<wire x1="22.86" y1="116.84" x2="20.32" y2="116.84" width="0.1524" layer="91"/>
+<label x="20.32" y="116.84" size="1.27" layer="95" ratio="10" rot="R180" xref="yes"/>
+</segment>
+</net>
+<net name="DIN" class="0">
+<segment>
+<pinref part="MOD1" gate="G$1" pin="D18/SCK"/>
+<wire x1="22.86" y1="104.14" x2="20.32" y2="104.14" width="0.1524" layer="91"/>
+<label x="20.32" y="104.14" size="1.27" layer="95" ratio="10" rot="R180" xref="yes"/>
+</segment>
+</net>
+<net name="CLK" class="0">
+<segment>
+<pinref part="MOD1" gate="G$1" pin="D19/MISO"/>
+<wire x1="22.86" y1="101.6" x2="20.32" y2="101.6" width="0.1524" layer="91"/>
+<label x="20.32" y="101.6" size="1.27" layer="95" ratio="10" rot="R180" xref="yes"/>
+</segment>
+</net>
+<net name="BL" class="0">
+<segment>
+<pinref part="MOD1" gate="G$1" pin="D21/SDA"/>
+<wire x1="22.86" y1="99.06" x2="20.32" y2="99.06" width="0.1524" layer="91"/>
+<label x="20.32" y="99.06" size="1.27" layer="95" ratio="10" rot="R180" xref="yes"/>
+</segment>
+</net>
+<net name="STATE" class="0">
+<segment>
+<pinref part="MOD1" gate="G$1" pin="D15/ADC2_3"/>
+<wire x1="22.86" y1="119.38" x2="20.32" y2="119.38" width="0.1524" layer="91"/>
+<label x="20.32" y="119.38" size="1.27" layer="95" ratio="10" rot="R180" xref="yes"/>
+</segment>
+</net>
+<net name="RXD2" class="0">
+<segment>
+<pinref part="MOD1" gate="G$1" pin="D16/RX2"/>
+<wire x1="22.86" y1="111.76" x2="20.32" y2="111.76" width="0.1524" layer="91"/>
+<label x="20.32" y="111.76" size="1.27" layer="95" ratio="10" rot="R180" xref="yes"/>
+</segment>
+</net>
+<net name="TXD2" class="0">
+<segment>
+<pinref part="MOD1" gate="G$1" pin="D17/TX2"/>
+<wire x1="22.86" y1="109.22" x2="20.32" y2="109.22" width="0.1524" layer="91"/>
+<label x="20.32" y="109.22" size="1.27" layer="95" ratio="10" rot="R180" xref="yes"/>
+</segment>
+</net>
+<net name="BOT-PANIC" class="0">
+<segment>
+<pinref part="MOD1" gate="G$1" pin="D14/ADC2_6"/>
+<wire x1="68.58" y1="114.3" x2="71.12" y2="114.3" width="0.1524" layer="91"/>
+<label x="71.12" y="114.3" size="1.27" layer="95" ratio="10" xref="yes"/>
+</segment>
+</net>
+<net name="DC" class="0">
+<segment>
+<pinref part="MOD1" gate="G$1" pin="D5"/>
+<wire x1="22.86" y1="106.68" x2="20.32" y2="106.68" width="0.1524" layer="91"/>
+<label x="20.32" y="106.68" size="1.27" layer="95" ratio="10" rot="R180" xref="yes"/>
+</segment>
+</net>
+<net name="CE" class="0">
+<segment>
+<pinref part="MOD1" gate="G$1" pin="D4/ADC2_0"/>
+<wire x1="22.86" y1="114.3" x2="20.32" y2="114.3" width="0.1524" layer="91"/>
+<label x="20.32" y="114.3" size="1.27" layer="95" ratio="10" rot="R180" xref="yes"/>
+</segment>
+</net>

Commit message: Terminado SCH y BRD
Parts:
- removed S1: (no value), adafruit:40-XX-ROUND
- removed X1: (no value), con-ptr500:AK500/2
- added C1: (no value), rcl:C-US050-025X075
- added R2: 1k, rcl:R-US_0204/7
- added S2: (no value), switch-omron:10-XX
Connections:
- net +3V3: now also S2.S, S2.S1
- net +5V: now also MOD2.+5V
- net BL: now also LCD1.BL
- net BOT-PANIC: now also C1.1, R1.1, S2.P, S2.P1
- net CE: now also LCD1.CE
- net CLK: now also LCD1.CLK
- net DC: now also LCD1.DC
- net DIN: now also LCD1.DIN
- net GND: now also C1.2, MOD2.GND, R1.2
- net LED: now also R2.1; no longer R1.1
- net N$1: now also R2.2; no longer R1.2
- net RST: now also LCD1.RST
- net RXD2: now also MOD2.TX
- net STATE: now also MOD2.STATE
- net TXD2: now also MOD2.RX
Other:
- note added: "MCU Y COMUNICACION WiFi"
- moved on the sheet: LCD1, MOD1, MOD2, R1
